File: HW/rf.kicad_sch (KiCad schematic)
At the start: 4 parts

Commit message: Almost first schematic draft (missing resistor values for STDRIVE current sensing and leds)
Parts:
- added AE1: Antenna_Shield, symbol Device:Antenna_Shield
- added C4: 0.4pF, Capacitor_SMD:C_0402_1005Metric, symbol Device:C
- added C5: 0.2pF, Capacitor_SMD:C_0402_1005Metric, symbol Device:C
- added C6, C7: ~, Capacitor_SMD:C_0402_1005Metric, symbol Device:C
- added R4: 0Ω, Resistor_SMD:R_0402_1005Metric, symbol Device:R
- C2, C3: footprint (none) -> Capacitor_SMD:C_0402_1005Metric
- L1: footprint (none) -> Inductor_SMD:L_0402_1005Metric
Connections:
- net GND: now also AE1.2 (Shield), C5.2, C6.2, C7.2
- net at FL1.3 (OUT): now also C4.2
- new net: C4.1, C7.1, R4.1
- new net: AE1.1 (A), C5.1, C6.1, R4.2
Other:
- note added: "Abracon PRO-OB-607 or similar?"
- note added: "Do we need an antenna matching circuit as well?"
- moved on the sheet: C2, C3, FL1, L1

Commit message: Cleaned up and implemented some of Laimonas' feedback
Other:
- note added: "Abracon PRO-OB-607 or similar"
- note removed: "Abracon PRO-OB-607 or similar?"
- note removed: "Do we need an antenna matching circuit as well?"
- company: (none) -> Roberto Holmes
- title: (none) -> Capstan
Changed lines of the file:
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@@
 	(generator_version "9.0")
 	(paper "A4")
-	(text "Abracon PRO-OB-607 or similar?"
+	(title_block
+		(title "Capstan")
+		(date "2025-09-26")
+		(company "Roberto Holmes")
+	)
+	(text "Abracon PRO-OB-607 or similar"
 		(exclude_from_sim no)
 		(at 194.056 70.358 0)
@@
 		)
 	)
-	(text "Do we need an antenna\nmatching circuit as well?"
-		(exclude_from_sim no)
-		(at 167.894 111.506 0)
-		(effects
-			(font
-				(size 1.27 1.27)
-			)
-		)
-	)
-	(text_box "TODO:\n- Is this antenna suitable?\n- Do we need two pi filters?\n- Are the pi filter values a good start point?\n- Do we need test points for calibration?"
-		(exclude_from_sim no)
-		(at 125.73 46.99 0)
-		(size 36.83 20.32)
-		(margins 0.9525 0.9525 0.9525 0.9525)
-		(stroke
-			(width 0)
-			(type solid)
-		)
-		(fill
-			(type none)
-		)
-		(effects
-			(font
-				(size 1.27 1.27)
-			)
-			(justify left top)
-		)
-	)
